File: Inett_60_PCB.kicad_pcb (KiCad board)
At the start: 2 copper layers, 158 parts, among them SW1 Reset, SW2 Boot, U1 RP2040, U2 W25Q128JVS, U3 XC6206PxxxMR, Y1 Crystal_GND24

Commit message: Add files via upload
Parts:
- C1, C10, C11, C12, C13, C14, C15, C16, C2, C3, C4, C5, C6, C7, C8, C9, C_S1, C_Shield1, D1, D10, D11, D12, D13, D14, D15, D16, D17, D18, D19, D2, D20, D21, D22, D23, D24, D25, D26, D27, D28, D29, D3, D30, D31, D32, D33, D34, D35, D36, D37, D38, D39, D4, D40, D41, D42, D43, D44, D45, D46, D47, D48, D49, D5, D50, D51, D52, D53, D54, D55, D56, D57, D58, D59, D6, D60, D61, D62, D7, D8, D9, R1, R2, R5, R6, R_Shield1, SW1, SW2, U1, U2, U3, Y1: moved to B.Cu
- D63, F1, MX1, MX10, MX11, MX12, MX13, MX14, MX15, MX16, MX17, MX18, MX19, MX2, MX20, MX21, MX22, MX23, MX24, MX25, MX26, MX27, MX28, MX29, MX3, MX30, MX31, MX32, MX33, MX34, MX35, MX36, MX37, MX38, MX39, MX4, MX40, MX41, MX42, MX43, MX44, MX45, MX46, MX47, MX48, MX49, MX5, MX50, MX51, MX52, MX53, MX54, MX55, MX56, MX57, MX58, MX59, MX6, MX60, MX61, MX62, MX7, MX8, MX9, R3, R4, USB1: moved to F.Cu
- moved D55 277.2 mm to (304.2, 97.6)
- moved D15 277.2 mm to (304.2, 40.6)
- moved D29 267.7 mm to (299.4, 59.6)
- moved D62 267.7 mm to (299.4, 116.6)
- moved MX15 267.1 mm to (299.1, 36.6), turned to 0 degrees
- moved MX55 267.1 mm to (299.1, 93.7), turned to 0 degrees
- moved MX1 266.3 mm to (32.4, 36.6), turned to 0 degrees
- moved MX29 257.6 mm to (294.3, 55.6), turned to 0 degrees
- moved MX62 257.6 mm to (294.3, 112.8), turned to 0 degrees
- moved MX16 256.8 mm to (37.1, 55.6), turned to 0 degrees
- moved MX56 256.8 mm to (37.1, 112.8), turned to 0 degrees
- moved D1 256.7 mm to (37.2, 40.6)
- moved D42 253.4 mm to (292.3, 78.6)
- moved MX30 252.0 mm to (39.5, 74.7), turned to 0 degrees
- moved D16 246.6 mm to (42.2, 59.6)
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Routing:
- added copper zone on F.Cu, net GND
- removed copper zone on B.Cu, net GND
